Commit message: 修正后评估测

File: isaaclab_logistics_vla/assets/robots/realman/realman_no_wheel.urdf (robot description, URDF)
Before this commit: robot realman_no_wheel, 24 links, 23 joints
Joints:
- joint right_left_joint: limit (none) -> lower=-6.28318530718 upper=6.28318530718 effort=10. velocity=5.
- joint right_right_joint: limit (none) -> lower=-6.28318530718 upper=6.28318530718 effort=10. velocity=5.
